File: PeltierArray/PeltierArray.kicad_pcb (KiCad board)
At the start: 2 copper layers, 1 part

Commit message: 玉巨的MOS
Parts:
- added CIN1: CP47uF, Capacitor_THT:C_Radial_D6.3mm_H11.0mm_P2.50mm, F.Cu at (91.0, 102.2)
- added CIN11: 47uF, Capacitor_SMD:C_1206_3216Metric, F.Cu at (99.2, 95.4)
- added CIN21: 1uF, Capacitor_SMD:C_0603_1608Metric, F.Cu at (102.4, 100.7)
- added COUT11: 10uF, Capacitor_SMD:C_0603_1608Metric, F.Cu at (98.8, 105.2)
- added COUT21: 1uF, Capacitor_SMD:C_0603_1608Metric, F.Cu at (98.8, 107.7)
- added DOUT1: D, Diode_SMD:D_SMA, F.Cu at (92.3, 96.0)
- added J1: Barrel_Jack, digikey-footprints:Barrel_Jack_5.5mmODx2.1mmID_PJ-102A, F.Cu at (83.0, 105.2)
- added LEDIN1: LED, LED:LED-0603, F.Cu at (98.1, 102.9)
- added LEDOUT1: LED, LED:LED-0603, F.Cu at (102.5, 98.1)
- added Peltier1: Conn_01x02_Male, Connector_JST:JST_PH_B2B-PH-K_1x02_P2.00mm_Vertical, F.Cu at (95.6, 77.4)
- added Q1: Q_NMOS_GDS, Package_TO_SOT_SMD:TO-252-2, F.Cu at (83.9, 77.8)
- added RIN1: 10K, Resistors:0603, F.Cu at (90.4, 107.3)
- added ROUT1: 10K, Resistors:0603, F.Cu at (98.5, 98.2)
- added RPWM11: 10, Resistors:0603, F.Cu at (98.3, 100.7)
- added RPWM21: 10K, Resistors:0603, F.Cu at (94.7, 107.3)
- added Temp1: Conn_01x02_Male, Connector_JST:JST_XH_B2B-XH-A_1x02_P2.50mm_Vertical, F.Cu at (81.3, 85.2)
Connections:
- MEGA2560PRO1 pad 3V3@1: (no net) -> +3V3
- MEGA2560PRO1 pad 3V3@2: (no net) -> +3V3
- MEGA2560PRO1 pad 5V@1: (no net) -> +5V
- MEGA2560PRO1 pad 5V@2: (no net) -> +5V
- MEGA2560PRO1 pad 5V@3: (no net) -> +5V
- MEGA2560PRO1 pad D2: (no net) -> /PWM1
- MEGA2560PRO1 pad GND@1: (no net) -> GND
- MEGA2560PRO1 pad GND@2: (no net) -> GND
- MEGA2560PRO1 pad GND@3: (no net) -> GND
- MEGA2560PRO1 pad VIN@1: (no net) -> +12V
- MEGA2560PRO1 pad VIN@2: (no net) -> +12V

Commit message: 玉巨溜了
Parts:
- J1: footprint digikey-footprints:Barrel_Jack_5.5mmODx2.1mmID_PJ-102A -> Connector_BarrelJack:BarrelJack_CUI_PJ-063AH_Horizontal
