File: PeltierArray/PeltierArray.sch (KiCad schematic (older format))
At the start: 1 part

Commit message: MOS
Parts:
- added J?: Conn_01x04_Male, Connector_JST:JST_PH_B4B-PH-SM4-TB_1x04-1MP_P2.00mm_Vertical, symbol Connector:Conn_01x04_Male
- added Q?: Q_NMOS_GDS, Package_TO_SOT_SMD:TO-252-2, symbol Device:Q_NMOS_GDS
Changed lines of the file:
@@
+	1    0    0    -1
+$EndComp
+$Comp
+L Connector:Conn_01x04_Male J?
+U 1 1 5F7F21F8
+P 6450 2000
+F 0 "J?" H 6558 2281 50  0000 C CNN
+F 1 "Conn_01x04_Male" H 6558 2190 50  0000 C CNN
+F 2 "Connector_JST:JST_PH_B4B-PH-SM4-TB_1x04-1MP_P2.00mm_Vertical" H 6450 2000 50  0001 C CNN
+F 3 "~" H 6450 2000 50  0001 C CNN
+	1    6450 2000
+	1    0    0    -1
+$EndComp
+$Comp
+L Device:Q_NMOS_GDS Q?
+U 1 1 5F7F3046
+P 7350 2350
+F 0 "Q?" H 7554 2396 50  0000 L CNN
+F 1 "Q_NMOS_GDS" H 7554 2305 50  0000 L CNN
+F 2 "Package_TO_SOT_SMD:TO-252-2" H 7550 2450 50  0001 C CNN
+F 3 "~" H 7350 2350 50  0001 C CNN
+	1    7350 2350
 	1    0    0    -1
 $EndComp

Commit message: 玉巨的MOS
Parts:
- removed J?: Conn_01x04_Male, Connector_JST:JST_PH_B4B-PH-SM4-TB_1x04-1MP_P2.00mm_Vertical, symbol Connector:Conn_01x04_Male
- added CIN: CP47uF, Capacitor_THT:C_Radial_D6.3mm_H11.0mm_P2.50mm, symbol Device:CP
- added CIN1?: 47uF, Capacitor_SMD:C_1206_3216Metric, symbol Device:C
- added CIN2?, COUT2?: 1uF, Capacitor_SMD:C_0603_1608Metric, symbol Device:C
- added COUT1?: 10uF, Capacitor_SMD:C_0603_1608Metric, symbol Device:C
- added DOUT?: D, Diode_SMD:D_SMA, symbol Device:D
- added J?: Barrel_Jack, digikey-footprints:Barrel_Jack_5.5mmODx2.1mmID_PJ-102A, symbol Connector:Barrel_Jack_MountingPin
- added LEDIN?, LEDOUT?: LED, LED:LED-0603, symbol Device:LED
- added Peltier?: Conn_01x02_Male, Connector_JST:JST_PH_B2B-PH-K_1x02_P2.00mm_Vertical, symbol Connector:Conn_01x02_Male
- added RIN?, ROUT?, RPWM2?: 10K, Resistors:0603, symbol Device:R
- added RPWM1?: 10, Resistors:0603, symbol Device:R
- added Temp?: Conn_01x02_Male, Connector_JST:JST_XH_B2B-XH-A_1x02_P2.50mm_Vertical, symbol Connector:Conn_01x02_Male
- gave numbers to parts that had none: 1
Connections:
- net +3V3: now reaches MEGA2560PRO1.3V3@1
- net +3V3: now also MEGA2560PRO1.3V3@2
- net +5V: now reaches MEGA2560PRO1.5V@1
- net +5V: now also MEGA2560PRO1.5V@2, MEGA2560PRO1.5V@3
- net PWM1: now reaches MEGA2560PRO1.D2
- net PWM1: now also RPWM1?.2, RPWM2?.2
- net GND: now reaches MEGA2560PRO1.GND@1
- net GND: now also MEGA2560PRO1.GND@2, MEGA2560PRO1.GND@3, Q1.3 (S), CIN.2, CIN1?.2, CIN2?.2, J?.2, J?.MP (MountPin), LEDIN?.1 (K), RPWM2?.1, Temp?.2 (Pin_2)
- net +12V: now reaches MEGA2560PRO1.VIN@1
- net +12V: now also MEGA2560PRO1.VIN@2
- net at Q1.1 (G): now also RPWM1?.1
- net at Q1.2 (D): now also COUT1?.2, COUT2?.2, DOUT?.2 (A), LEDOUT?.1 (K), Peltier?.2 (Pin_2)
- new net: LEDOUT?.2 (A), ROUT?.2
- new net: LEDIN?.2 (A), RIN?.2
- new net +BATT: CIN.1, CIN1?.1, CIN2?.1, COUT1?.1, COUT2?.1, DOUT?.1 (K), J?.1, Peltier?.1 (Pin_1), RIN?.1, ROUT?.1
- new net Temp1: Temp?.1 (Pin_1)
Other:
- moved on the sheet: MEGA2560PRO1, Q1

Commit message: 玉巨溜了
Parts:
- J?: footprint digikey-footprints:Barrel_Jack_5.5mmODx2.1mmID_PJ-102A -> Connector_BarrelJack:BarrelJack_Wuerth_6941xx301002
- gave numbers to parts that had none: 6
- renumbered CIN to CIN?, MEGA2560PRO1 to MEGA2560PRO?, Q1 to Q?
Connections:
- net Temp1: now also MEGA2560PRO?.A0
Other:
- moved on the sheet: CIN?, COUT?, DOUT?, J?, LEDIN?, LEDOUT?, MEGA2560PRO?, Peltier?, Q?, RIN?, ROUT?, RPWM?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

Commit message: Add Filter Temp Sensor
Parts:
- added CTemp?: 100nF, Capacitor_SMD:C_0603_1608Metric, symbol Device:C
- added RTemp?: 500, Resistors:0603, symbol Device:R
Connections:
- net GND: now also CTemp?.2
- net Temp1: now also CTemp?.1, RTemp?.1; no longer Temp?.1 (Pin_1)
- new net: RTemp?.2, Temp?.1 (Pin_1)
Changed lines of the file:
@@
 L power:GND #PWR?
 U 1 1 5F866984
-P 7200 5700
-F 0 "#PWR?" H 7200 5450 50  0001 C CNN
-F 1 "GND" H 7205 5527 50  0000 C CNN
-F 2 "" H 7200 5700 50  0001 C CNN
-F 3 "" H 7200 5700 50  0001 C CNN
-	1    7200 5700
+P 7200 6050
+F 0 "#PWR?" H 7200 5800 50  0001 C CNN
+F 1 "GND" H 7205 5877 50  0000 C CNN
+F 2 "" H 7200 6050 50  0001 C CNN
+F 3 "" H 7200 6050 50  0001 C CNN
+	1    7200 6050
 	1    0    0    -1
 $EndComp
 Wire Wire Line
 	7100 5600 7200 5600
-Wire Wire Line
-	7200 5600 7200 5700
-Wire Wire Line
-	7100 5500 7400 5500
-Text Label 7400 5500 0    50   ~ 0
+Text Label 7950 5500 0    50   ~ 0
 Temp1
 $Comp
@@
 Text Label 6150 4650 0    50   ~ 0
 Temp1
+$Comp
+L Device:R RTemp?
+U 1 1 5F7FEA2A
+P 7500 5500
+F 0 "RTemp?" H 7430 5454 50  0000 R CNN
+F 1 "500" H 7430 5545 50  0000 R CNN
+F 2 "Resistors:0603" V 7430 5500 50  0001 C CNN
+F 3 "~" H 7500 5500 50  0001 C CNN
+	1    7500 5500
+	0    1    1    0
+$EndComp
+$Comp
+L Device:C CTemp?
+U 1 1 5F7FF4CF
+P 7800 5700
+F 0 "CTemp?" H 7915 5746 50  0000 L CNN
+F 1 "100nF" H 7915 5655 50  0000 L CNN
+F 2 "Capacitor_SMD:C_0603_1608Metric" H 7838 5550 50  0001 C CNN
+F 3 "~" H 7800 5700 50  0001 C CNN
+	1    7800 5700
+	1    0    0    -1
+$EndComp
+Wire Wire Line
+	7650 5500 7800 5500
+Wire Wire Line
+	7800 5550 7800 5500
+Connection ~ 7800 5500
+Wire Wire Line
+	7800 5500 7950 5500
+Wire Wire Line
+	7800 5900 7800 5850
+Wire Wire Line
+	7200 5600 7200 5900
+Wire Wire Line
+	7100 5500 7350 5500
+Wire Wire Line
+	7800 5900 7200 5900
+Connection ~ 7200 5900
+Wire Wire Line
+	7200 5900 7200 6050
 $EndSCHEMATC

Commit message: 热敏电阻
Parts:
- removed RTemp?: 500, Resistors:0603, symbol Device:R
- added RTemp?: 10K, Resistors:0603, symbol Device:R
Connections:
- net +5V: now also CTemp?.1, Temp?.1 (Pin_1)
- net GND: now also RTemp?.1; no longer Temp?.2 (Pin_2)
- net Temp1: now also Temp?.2 (Pin_2), RTemp?.2; no longer CTemp?.1
Other:
- moved on the sheet: CTemp?, Temp?
Changed lines of the file:
@@
 L Connector:Conn_01x02_Male Temp?
 U 1 1 5F7FC7AE
-P 6900 5500
-F 0 "Temp?" H 7008 5681 50  0000 C CNN
-F 1 "Conn_01x02_Male" H 7008 5590 50  0000 C CNN
-F 2 "Connector_JST:JST_XH_B2B-XH-A_1x02_P2.50mm_Vertical" H 6900 5500 50  0001 C CNN
-F 3 "~" H 6900 5500 50  0001 C CNN
-	1    6900 5500
+P 1550 1600
+F 0 "Temp?" H 1658 1781 50  0000 C CNN
+F 1 "Conn_01x02_Male" H 1658 1690 50  0000 C CNN
+F 2 "Connector_JST:JST_XH_B2B-XH-A_1x02_P2.50mm_Vertical" H 1550 1600 50  0001 C CNN
+F 3 "~" H 1550 1600 50  0001 C CNN
+	1    1550 1600
 	1    0    0    -1
 $EndComp
@@
 L power:GND #PWR?
 U 1 1 5F866984
-P 7200 6050
-F 0 "#PWR?" H 7200 5800 50  0001 C CNN
-F 1 "GND" H 7205 5877 50  0000 C CNN
-F 2 "" H 7200 6050 50  0001 C CNN
-F 3 "" H 7200 6050 50  0001 C CNN
-	1    7200 6050
-	1    0    0    -1
-$EndComp
-Wire Wire Line
-	7100 5600 7200 5600
-Text Label 7950 5500 0    50   ~ 0
+P 1750 2300
+F 0 "#PWR?" H 1750 2050 50  0001 C CNN
+F 1 "GND" H 1755 2127 50  0000 C CNN
+F 2 "" H 1750 2300 50  0001 C CNN
+F 3 "" H 1750 2300 50  0001 C CNN
+	1    1750 2300
+	1    0    0    -1
+$EndComp
+Text Label 1250 1850 0    50   ~ 0
 Temp1
 $Comp
@@
 Temp1
 $Comp
-L Device:R RTemp?
-U 1 1 5F7FEA2A
-P 7500 5500
-F 0 "RTemp?" H 7430 5454 50  0000 R CNN
-F 1 "500" H 7430 5545 50  0000 R CNN
-F 2 "Resistors:0603" V 7430 5500 50  0001 C CNN
-F 3 "~" H 7500 5500 50  0001 C CNN
-	1    7500 5500
-	0    1    1    0
-$EndComp
-$Comp
 L Device:C CTemp?
 U 1 1 5F7FF4CF
-P 7800 5700
-F 0 "CTemp?" H 7915 5746 50  0000 L CNN
-F 1 "100nF" H 7915 5655 50  0000 L CNN
-F 2 "Capacitor_SMD:C_0603_1608Metric" H 7838 5550 50  0001 C CNN
-F 3 "~" H 7800 5700 50  0001 C CNN
-	1    7800 5700
-	1    0    0    -1
-$EndComp
-Wire Wire Line
-	7650 5500 7800 5500
-Wire Wire Line
-	7800 5550 7800 5500
-Connection ~ 7800 5500
-Wire Wire Line
-	7800 5500 7950 5500
-Wire Wire Line
-	7800 5900 7800 5850
-Wire Wire Line
-	7200 5600 7200 5900
-Wire Wire Line
-	7100 5500 7350 5500
-Wire Wire Line
-	7800 5900 7200 5900
-Connection ~ 7200 5900
-Wire Wire Line
-	7200 5900 7200 6050
+P 2200 1700
+F 0 "CTemp?" H 2315 1746 50  0000 L CNN
+F 1 "100nF" H 2315 1655 50  0000 L CNN
+F 2 "Capacitor_SMD:C_0603_1608Metric" H 2238 1550 50  0001 C CNN
+F 3 "~" H 2200 1700 50  0001 C CNN
+	1    2200 1700
+	1    0    0    -1
+$EndComp
+$Comp
+L Device:R RTemp?
+U 1 1 5F826DF9
+P 1750 2050
+F 0 "RTemp?" H 1680 2004 50  0000 R CNN
+F 1 "10K" H 1680 2095 50  0000 R CNN
+F 2 "Resistors:0603" V 1680 2050 50  0001 C CNN
+F 3 "~" H 1750 2050 50  0001 C CNN
+	1    1750 2050
+	-1   0    0    1
+$EndComp
+Wire Wire Line
+	1750 1850 1750 1900
+Wire Wire Line
+	1250 1850 1750 1850
+$Comp
+L power:+5V #PWR?
+U 1 1 5F83597C
+P 1750 1300
+F 0 "#PWR?" H 1750 1150 50  0001 C CNN
+F 1 "+5V" V 1765 1428 50  0000 L CNN
+F 2 "" H 1750 1300 50  0001 C CNN
+F 3 "" H 1750 1300 50  0001 C CNN
+	1    1750 1300
+	1    0    0    -1
+$EndComp
+Wire Wire Line
+	1750 2200 1750 2250
+Wire Wire Line
+	1750 1300 1750 1350
+Wire Wire Line
+	1750 1700 1750 1850
+Connection ~ 1750 1850
+Wire Wire Line
+	1750 2250 2200 2250
+Wire Wire Line
+	2200 2250 2200 1850
+Connection ~ 1750 2250
+Wire Wire Line
+	1750 2250 1750 2300
+Wire Wire Line
+	1750 1350 2200 1350
+Wire Wire Line
+	2200 1350 2200 1550
+Connection ~ 1750 1350
+Wire Wire Line
+	1750 1350 1750 1600
 $EndSCHEMATC
