File: PeltierArray-V2/TB6612.sch (KiCad schematic (older format))
At the start: 3 parts

Commit message: UART I2C
Parts:
- added CTemp10, CTemp9: 100nF, Capacitor_SMD:C_0603_1608Metric, symbol Device:C
- added RTemp10, RTemp9: 10K, Resistors:0603, symbol Device:R
- added Temp10, Temp9: Conn_01x02_Male, Connector_JST:JST_XH_B2B-XH-A_1x02_P2.50mm_Vertical, symbol Connector:Conn_01x02_Male
- renumbered Peltier2 to Peltier10, Peltier1 to Peltier9, TB6612FNG1 to TB6612FNG5
Connections:
- net +5V: now also CTemp10.1, CTemp9.1, Temp10.1 (Pin_1), Temp9.1 (Pin_1)
- net GND: now also CTemp10.2, CTemp9.2, RTemp10.1, RTemp9.1
- new net TempA: RTemp9.2, Temp9.2 (Pin_2)
- new net TempB: RTemp10.2, Temp10.2 (Pin_2)
Other:
- moved on the sheet: Peltier10, Peltier9, TB6612FNG5

Commit message: BeginRoute
Parts:
- Peltier10, Peltier9: footprint Connector_JST:JST_PH_B2B-PH-K_1x02_P2.00mm_Vertical -> Connector_JST:JST_XH_B2B-XH-A_1x02_P2.50mm_Vertical
Changed lines of the file:
@@
 $Descr A4 11693 8268
 encoding utf-8
-Sheet 6 6
+Sheet 5 6
 Title ""
 Date ""
@@
 F 0 "Peltier10" H 3258 3631 50  0000 C CNN
 F 1 "Conn_01x02_Male" H 3258 3540 50  0000 C CNN
-F 2 "Connector_JST:JST_PH_B2B-PH-K_1x02_P2.00mm_Vertical" H 3150 3450 50  0001 C CNN
+F 2 "Connector_JST:JST_XH_B2B-XH-A_1x02_P2.50mm_Vertical" H 3150 3450 50  0001 C CNN
 F 3 "~" H 3150 3450 50  0001 C CNN
 	1    3150 3450
@@
 F 0 "Peltier9" H 3258 3181 50  0000 C CNN
 F 1 "Conn_01x02_Male" H 3258 3090 50  0000 C CNN
-F 2 "Connector_JST:JST_PH_B2B-PH-K_1x02_P2.00mm_Vertical" H 3150 3000 50  0001 C CNN
+F 2 "Connector_JST:JST_XH_B2B-XH-A_1x02_P2.50mm_Vertical" H 3150 3000 50  0001 C CNN
 F 3 "~" H 3150 3000 50  0001 C CNN
 	1    3150 3000

Commit message: FUUUUUUCK
Parts:
- renumbered CTemp9 to CTemp10, CTemp10 to CTemp9, RTemp9 to RTemp10, RTemp10 to RTemp9, Temp9 to Temp10, Temp10 to Temp9
