File: PeltierArray-V3/PeltierArray.sch (KiCad schematic (older format))
At the start: 17 parts, among them J1 Barrel_Jack

Commit message: V3Finish
Parts:
- L1, L2: footprint Inductor_SMD:L_Taiyo-Yuden_NR-60xx_HandSoldering -> Inductor_SMD:L_Wuerth_HCM-1390
Changed lines of the file:
@@
 F 0 "L1" V 8340 3150 50  0000 C CNN
 F 1 "L 33uF 4.5A" V 8249 3150 50  0000 C CNN
-F 2 "Inductor_SMD:L_Taiyo-Yuden_NR-60xx_HandSoldering" H 8150 3150 50  0001 C CNN
+F 2 "Inductor_SMD:L_Wuerth_HCM-1390" H 8150 3150 50  0001 C CNN
 F 3 "~" H 8150 3150 50  0001 C CNN
 	1    8150 3150
@@
 F 0 "L2" V 8340 4550 50  0000 C CNN
 F 1 "L 33uF 4.5A" V 8249 4550 50  0000 C CNN
-F 2 "Inductor_SMD:L_Taiyo-Yuden_NR-60xx_HandSoldering" H 8150 4550 50  0001 C CNN
+F 2 "Inductor_SMD:L_Wuerth_HCM-1390" H 8150 4550 50  0001 C CNN
 F 3 "~" H 8150 4550 50  0001 C CNN
 	1    8150 4550
