File: PeltierArray-V3/TB6612.sch (KiCad schematic (older format))
At the start: 9 parts

Commit message: V3Finish
Changed lines of the file:
@@
 $Descr A4 11693 8268
 encoding utf-8
-Sheet 4 6
+Sheet 6 6
 Title ""
 Date ""
@@
 AR Path="/5F8773C4/5F8A1F60" Ref="TB6612FNG?"  Part="1"
 AR Path="/5F8773D8/5F8A1F60" Ref="TB6612FNG?"  Part="1"
-F 0 "TB6612FNG3" H 4400 4815 50  0000 C CNN
+F 0 "TB6612FNG5" H 4400 4815 50  0000 C CNN
 F 1 "TB6612FNG" H 4400 4724 50  0000 C CNN
 F 2 "PeltierArray:DIP-16_617_ELL" H 4400 3700 50  0001 C CNN
@@
 AR Path="/5F8773C4/5F8A1F66" Ref="Peltier?"  Part="1"
 AR Path="/5F8773D8/5F8A1F66" Ref="Peltier?"  Part="1"
-F 0 "Peltier6" H 3258 3631 50  0000 C CNN
+F 0 "Peltier10" H 3258 3631 50  0000 C CNN
 F 1 "Conn_01x02_Male" H 3258 3540 50  0000 C CNN
 F 2 "Connector_JST:JST_XH_B2B-XH-A_1x02_P2.50mm_Vertical" H 3150 3450 50  0001 C CNN
@@
 AR Path="/5F8773C4/5F8A1FA8" Ref="Peltier?"  Part="1"
 AR Path="/5F8773D8/5F8A1FA8" Ref="Peltier?"  Part="1"
-F 0 "Peltier5" H 3258 3181 50  0000 C CNN
+F 0 "Peltier9" H 3258 3181 50  0000 C CNN
 F 1 "Conn_01x02_Male" H 3258 3090 50  0000 C CNN
 F 2 "Connector_JST:JST_XH_B2B-XH-A_1x02_P2.50mm_Vertical" H 3150 3000 50  0001 C CNN
@@
 AR Path="/5F8695C5/5F90713C" Ref="Temp6"  Part="1"
 AR Path="/5F85874B/5F90713C" Ref="Temp8"  Part="1"
-F 0 "Temp6" H 6308 3131 50  0000 C CNN
+F 0 "Temp10" H 6308 3131 50  0000 C CNN
 F 1 "Conn_01x02_Male" H 6308 3040 50  0000 C CNN
 F 2 "Connector_JST:JST_XH_B2B-XH-A_1x02_P2.50mm_Vertical" H 6200 2950 50  0001 C CNN
@@
 AR Path="/5F8695C5/5F907149" Ref="CTemp6"  Part="1"
 AR Path="/5F85874B/5F907149" Ref="CTemp8"  Part="1"
-F 0 "CTemp6" H 6965 3096 50  0000 L CNN
+F 0 "CTemp10" H 6965 3096 50  0000 L CNN
 F 1 "100nF" H 6965 3005 50  0000 L CNN
 F 2 "Capacitor_SMD:C_0603_1608Metric" H 6888 2900 50  0001 C CNN
@@
 AR Path="/5F8695C5/5F90714F" Ref="RTemp6"  Part="1"
 AR Path="/5F85874B/5F90714F" Ref="RTemp8"  Part="1"
-F 0 "RTemp6" H 6330 3354 50  0000 R CNN
+F 0 "RTemp10" H 6330 3354 50  0000 R CNN
 F 1 "10K" H 6330 3445 50  0000 R CNN
 F 2 "Resistors:0603" V 6330 3400 50  0001 C CNN
@@
 AR Path="/5F8695C5/5F90DD09" Ref="Temp5"  Part="1"
 AR Path="/5F85874B/5F90DD09" Ref="Temp7"  Part="1"
-F 0 "Temp5" H 7958 3081 50  0000 C CNN
+F 0 "Temp9" H 7958 3081 50  0000 C CNN
 F 1 "Conn_01x02_Male" H 7958 2990 50  0000 C CNN
 F 2 "Connector_JST:JST_XH_B2B-XH-A_1x02_P2.50mm_Vertical" H 7850 2900 50  0001 C CNN
@@
 AR Path="/5F8695C5/5F90DD15" Ref="CTemp5"  Part="1"
 AR Path="/5F85874B/5F90DD15" Ref="CTemp7"  Part="1"
-F 0 "CTemp5" H 8615 3046 50  0000 L CNN
+F 0 "CTemp9" H 8615 3046 50  0000 L CNN
 F 1 "100nF" H 8615 2955 50  0000 L CNN
 F 2 "Capacitor_SMD:C_0603_1608Metric" H 8538 2850 50  0001 C CNN
@@
 AR Path="/5F8695C5/5F90DD1B" Ref="RTemp5"  Part="1"
 AR Path="/5F85874B/5F90DD1B" Ref="RTemp7"  Part="1"
-F 0 "RTemp5" H 7980 3304 50  0000 R CNN
+F 0 "RTemp9" H 7980 3304 50  0000 R CNN
 F 1 "10K" H 7980 3395 50  0000 R CNN
 F 2 "Resistors:0603" V 7980 3350 50  0001 C CNN
